Commit message: over

File: arm_description/urdf/arm_description.urdf (robot description, URDF)
Before this commit: robot arm_description, 9 links, 8 joints
Links:
- added link base_footprint
Joints:
- added joint base_footprint_joint: type fixed, parent base_footprint, child base_link, origin xyz=0 0 0.001 rpy=0 0 0
